Commit message: Add validated HC10 perception and pick-place integration

File: src/hc10_moveit_config/urdf/hc10_mfja.urdf.xacro (robot description, xacro)
@@ -4,6 +4,6 @@
   <xacro:macro name="mesh_link" params="name mesh">
     <link name="${name}">
-      <visual><geometry><mesh filename="package://motoman_hc10_support/meshes/hc10/visual/${mesh}.dae"/></geometry><material name="yaskawa_blue"/></visual>
-      <collision><geometry><mesh filename="package://motoman_hc10_support/meshes/hc10/collision/${mesh}.stl"/></geometry></collision>
+      <visual><geometry><mesh filename="package://mfja_3rd_floor_description/models/yaskawa_hc10/meshes/hc10/visual/${mesh}.dae"/></geometry><material name="yaskawa_blue"/></visual>
+      <collision><geometry><mesh filename="package://mfja_3rd_floor_description/models/yaskawa_hc10/meshes/hc10/collision/${mesh}.stl"/></geometry></collision>
     </link>
   </xacro:macro>
@@ -15,10 +15,10 @@
   </xacro:macro>
   <xacro:mesh_link name="base_link" mesh="base_link"/>
-  <xacro:mesh_link name="link_1_s" mesh="link_1"/>
-  <xacro:mesh_link name="link_2_l" mesh="link_2"/>
-  <xacro:mesh_link name="link_3_u" mesh="link_3"/>
-  <xacro:mesh_link name="link_4_r" mesh="link_4"/>
-  <xacro:mesh_link name="link_5_b" mesh="link_5"/>
-  <xacro:mesh_link name="link_6_t" mesh="link_6"/>
+  <xacro:mesh_link name="link_1_s" mesh="link_1_s"/>
+  <xacro:mesh_link name="link_2_l" mesh="link_2_l"/>
+  <xacro:mesh_link name="link_3_u" mesh="link_3_u"/>
+  <xacro:mesh_link name="link_4_r" mesh="link_4_r"/>
+  <xacro:mesh_link name="link_5_b" mesh="link_5_b"/>
+  <xacro:mesh_link name="link_6_t" mesh="link_6_t"/>
   <xacro:arm_joint name="joint_1_s" parent="base_link" child="link_1_s" xyz="0 0 0.275" axis="0 0 1" lower="-${pi}" upper="${pi}" effort="368.48" velocity="2.26892802759"/>
   <xacro:arm_joint name="joint_2_l" parent="link_1_s" child="link_2_l" xyz="0 0 0" axis="0 1 0" lower="-${pi}" upper="${pi}" effort="368.48" velocity="2.26892802759"/>
@@ -31,4 +31,20 @@
   <link name="gripper"><visual><origin xyz="0 0 0.024"/><geometry><box size="0.090 0.078 0.048"/></geometry></visual><collision><origin xyz="0 0 0.024"/><geometry><box size="0.090 0.078 0.048"/></geometry></collision></link>
   <joint name="tool0-gripper" type="fixed"><parent link="tool0"/><child link="gripper"/></joint>
+  <link name="gripper_left_jaw">
+    <visual><origin xyz="0.0075 0 0.0525"/><geometry><box size="0.004 0.019 0.035"/></geometry></visual>
+    <collision><origin xyz="0.0075 0 0.0525"/><geometry><box size="0.004 0.019 0.035"/></geometry></collision>
+  </link>
+  <joint name="gripper_left_jaw_joint" type="prismatic">
+    <origin xyz="-0.025 0 0.0482"/><parent link="gripper"/><child link="gripper_left_jaw"/>
+    <axis xyz="-1 0 0"/><limit lower="0" upper="0.040" effort="80" velocity="0.06"/>
+  </joint>
+  <link name="gripper_right_jaw">
+    <visual><origin xyz="-0.0075 0 0.0525"/><geometry><box size="0.004 0.019 0.035"/></geometry></visual>
+    <collision><origin xyz="-0.0075 0 0.0525"/><geometry><box size="0.004 0.019 0.035"/></geometry></collision>
+  </link>
+  <joint name="gripper_right_jaw_joint" type="prismatic">
+    <origin xyz="0.025 0 0.0482"/><parent link="gripper"/><child link="gripper_right_jaw"/>
+    <axis xyz="1 0 0"/><limit lower="0" upper="0.040" effort="80" velocity="0.06"/>
+  </joint>
   <link name="gripper_tcp"/>
   <joint name="gripper_tcp_joint" type="fixed"><origin xyz="0 0 0.1182"/><parent link="gripper"/><child link="gripper_tcp"/></joint>

Commit message: Ajout de la commande HC10 par pose

File: src/hc10_moveit_config/urdf/hc10_mfja.urdf.xacro (robot description, xacro)
@@ -4,6 +4,6 @@
   <xacro:macro name="mesh_link" params="name mesh">
     <link name="${name}">
-      <visual><geometry><mesh filename="package://motoman_hc10_support/meshes/hc10/visual/${mesh}.dae"/></geometry><material name="yaskawa_blue"/></visual>
-      <collision><geometry><mesh filename="package://motoman_hc10_support/meshes/hc10/collision/${mesh}.stl"/></geometry></collision>
+      <visual><geometry><mesh filename="package://mfja_3rd_floor_description/models/yaskawa_hc10/meshes/hc10/visual/${mesh}.dae"/></geometry><material name="yaskawa_blue"/></visual>
+      <collision><geometry><mesh filename="package://mfja_3rd_floor_description/models/yaskawa_hc10/meshes/hc10/collision/${mesh}.stl"/></geometry></collision>
     </link>
   </xacro:macro>
@@ -15,10 +15,10 @@
   </xacro:macro>
   <xacro:mesh_link name="base_link" mesh="base_link"/>
-  <xacro:mesh_link name="link_1_s" mesh="link_1"/>
-  <xacro:mesh_link name="link_2_l" mesh="link_2"/>
-  <xacro:mesh_link name="link_3_u" mesh="link_3"/>
-  <xacro:mesh_link name="link_4_r" mesh="link_4"/>
-  <xacro:mesh_link name="link_5_b" mesh="link_5"/>
-  <xacro:mesh_link name="link_6_t" mesh="link_6"/>
+  <xacro:mesh_link name="link_1_s" mesh="link_1_s"/>
+  <xacro:mesh_link name="link_2_l" mesh="link_2_l"/>
+  <xacro:mesh_link name="link_3_u" mesh="link_3_u"/>
+  <xacro:mesh_link name="link_4_r" mesh="link_4_r"/>
+  <xacro:mesh_link name="link_5_b" mesh="link_5_b"/>
+  <xacro:mesh_link name="link_6_t" mesh="link_6_t"/>
   <xacro:arm_joint name="joint_1_s" parent="base_link" child="link_1_s" xyz="0 0 0.275" axis="0 0 1" lower="-${pi}" upper="${pi}" effort="368.48" velocity="2.26892802759"/>
   <xacro:arm_joint name="joint_2_l" parent="link_1_s" child="link_2_l" xyz="0 0 0" axis="0 1 0" lower="-${pi}" upper="${pi}" effort="368.48" velocity="2.26892802759"/>
